Commit message: Added data2 inside the git repo

File: scenes/g500ARMPandora.urdf (robot description, URDF)
Before this commit: robot girona500, 7 links, 6 joints
Links:
- link base_link: geometry visual mesh filename=package://udg_pandora/data2/robot2/GIRONA500v2/g500.osg

Commit message: Added the new arm for the PANDORA PROJECT.
Forward and Inverse Kinematics are operative
The frame used is respect of the arm, not from the robot.
Will be fixed soon.

The movement of the arm is not really smooth in the trajectories.
Soon Will be working.

File: scenes/g500ARMPandora.urdf (robot description, URDF)
Before this commit: robot girona500, 7 links, 6 joints
Links:
- removed link arm
- removed link hand
- removed link jaw1
- removed link jaw2
- removed link support
- added link biceps; visual mesh filename=package://udg_pandora/data2/robot2/NEW_PANDORA_ARM/part3.osg
- added link forearm; visual mesh filename=package://udg_pandora/data2/robot2/NEW_PANDORA_ARM/part4.osg
- added link jawI; visual mesh filename=package://udg_pandora/data2/robot2/NEW_PANDORA_ARM/jawI.osg
- added link jawS; visual mesh filename=package://udg_pandora/data2/robot2/NEW_PANDORA_ARM/jawS.osg
- added link palm; visual mesh filename=package://udg_pandora/data2/robot2/NEW_PANDORA_ARM/part5.osg
- added link shoulder; visual mesh filename=package://udg_pandora/data2/robot2/NEW_PANDORA_ARM/part2.osg
- link base: geometry visual mesh filename=package://udg_pandora/data2/robot2/NEW_PANDORA_ARM/part1.osg
Joints:
- removed joint arm_to_hand
- removed joint base_to_arm
- removed joint hand_to_support
- removed joint support_to_jaw1
- added joint base_to_shoulder: type continuous, parent base, child shoulder, origin xyz=0.25 -0.02 0.0 rpy=0 0 0, axis 0 0 1
- added joint elbow: type continuous, parent biceps, child forearm, origin xyz=0.22 0.0 0.05 rpy=0 0 0, axis 0 1 0
- added joint palm_to_jawS: type continuous, parent palm, child jawS, origin xyz=0.08 0.03 0.0 rpy=0 0 0.5, axis 0 0 1
- added joint shoulder_to_biceps: type continuous, parent shoulder, child biceps, origin xyz=0.10 0.0 0.05 rpy=0 0 0, axis 0 1 0
- added joint wrist: type continuous, parent forearm, child palm, origin xyz=0.2 0.01 -0.1 rpy=0 0 0, axis 1 0 0
- joint baselink_to_base: origin xyz=0.5 0.0 0.77 rpy=0 0 0 -> xyz=0.5 0.0 0.75 rpy=0 0 0
- joint support_to_jaw2: axis 0 1 0 -> 0 0 -1; child jaw2 -> jawI; mimic joint=support_to_jaw1 multiplier=1 offset=0 -> joint=palm_to_jawS multiplier=1 offset=0; origin xyz=0.12 0 0.0 rpy=0 0 0 -> xyz=0.08 -0.03 0.0 rpy=0 0 -0.5; parent support -> palm; type fixed -> continuous

Commit message: Changed the Mesh of the G500. The center of the mesh is equal with the center of the real vehicle

File: scenes/g500ARMPandora.urdf (robot description, URDF)
Before this commit: robot girona500, 8 links, 7 joints
Joints:
- joint baselink_to_base: origin xyz=0.5 0.0 0.75 rpy=0 0 0 -> xyz=0.5 0.0 0.4 rpy=0 0 0

Commit message: Added a new Controller for shared movement between arm and vehicle

File: scenes/g500ARMPandora.urdf (robot description, URDF)
Before this commit: robot girona500, 8 links, 7 joints
Joints:
- joint elbow: origin xyz=0.22 0.0 0.05 rpy=0 0 0 -> xyz=0.22 0.0 0.05 rpy=0 -1.57 0
- joint shoulder_to_biceps: origin xyz=0.10 0.0 0.05 rpy=0 0 0 -> xyz=0.10 0.0 0.0 rpy=0 0 0
