Commit message: Added the new panel with one handle

File: scenes/valvePanel.urdf (robot description, URDF)
Before this commit: robot valvePanel, 7 links, 6 joints
Links:
- removed link handle01
- removed link handle02
- removed link handle03
- removed link handle04
- removed link handle05
- removed link handle06
- removed link panel
- added link bar; visual mesh filename=package://udg_pandora/data2/objects2/handle.osg
- added link handle; visual mesh filename=package://udg_pandora/data2/objects2/handle.osg
Joints:
- removed joint panel_to_handle_01
- removed joint panel_to_handle_02
- removed joint panel_to_handle_03
- removed joint panel_to_handle_04
- removed joint panel_to_handle_05
- removed joint panel_to_handle_06
- added joint valve: type continuous, parent bar, child handle, origin xyz=0.05 0.01 0.0 rpy=0 0 0, axis 1 0 0
