Commit message: iit staff

File: scenes/g500ARMPandora_backUp.urdf (robot description, URDF)
Before this commit: robot girona500, 10 links, 9 joints
Links:
- removed link virtual_wrist_1
- removed link virtual_wrist_2
Joints:
- removed joint virtual_wrist_roll
- removed joint virtual_wrist_roll_2
- joint base_to_shoulder: limit lower=-0.52 upper=1.57 effort=1000.0 velocity=0.733 -> (none); type revolute -> continuous
- joint elbow: limit lower=-3.14 upper=-0.82 effort=1000.0 velocity=0.733 -> (none); origin xyz=0.22 0.0 0.05 rpy=0 0 0 -> xyz=0.22 0.0 0.05 rpy=0 -1.57 0; type revolute -> continuous
- joint shoulder_to_biceps: limit lower=0.0 upper=1.57 effort=1000.0 velocity=0.733 -> (none); origin xyz=0.10 0.0 0.05 rpy=0 0 0 -> xyz=0.10 0.0 0.0 rpy=0 0 0; type revolute -> continuous
- joint wrist: parent virtual_wrist_2 -> forearm
