Commit message: Added important stuff

File: scenes/g500ARMPandora_iit.urdf (robot description, URDF)
Before this commit: robot girona500, 8 links, 7 joints
Links:
- added link virtual_wrist_1; visual cylinder length=0.0 radius=0.0
- added link virtual_wrist_2; visual cylinder length=0.0 radius=0.0
Joints:
- added joint virtual_wrist_roll: type continuous, parent forearm, child virtual_wrist_1, axis 0 1 0
- added joint virtual_wrist_roll_2: type continuous, parent virtual_wrist_1, child virtual_wrist_2, axis 0 0 1
- joint base_to_shoulder: limit (none) -> lower=-0.52 upper=1.57 effort=1000.0 velocity=0.733; type continuous -> revolute
- joint elbow: limit (none) -> lower=-3.14 upper=-0.82 effort=1000.0 velocity=0.733; origin xyz=0.22 0.0 0.05 rpy=0 -1.57 0 -> xyz=0.22 0.0 0.05 rpy=0 0 0; type continuous -> revolute
- joint shoulder_to_biceps: limit (none) -> lower=0.0 upper=1.57 effort=1000.0 velocity=0.733; origin xyz=0.10 0.0 0.0 rpy=0 0 0 -> xyz=0.10 0.0 0.05 rpy=0 0 0; type continuous -> revolute
- joint wrist: parent forearm -> virtual_wrist_2
