Commit message: Reorganize udg_pandora package in sub packages

File: udg_pandora_sim/scenes/g500ARMPandora.urdf (robot description, URDF)
Before this commit: robot girona500, 8 links, 7 joints
Links:
- link base: geometry visual mesh filename=package://udg_pandora_sim/data2/robot2/NEW_PANDORA_ARM/part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
- link base_link: geometry visual mesh filename=package://udg_pandora_sim/data2/robot2/GIRONA500v2/g500.osg
- link biceps: geometry visual mesh filename=package://udg_pandora_sim/data2/robot2/NEW_PANDORA_ARM/part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
- link forearm: geometry visual mesh filename=package://udg_pandora_sim/data2/robot2/NEW_PANDORA_ARM/part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
- link jawI: geometry visual mesh filename=package://udg_pandora_sim/data2/robot2/NEW_PANDORA_ARM/jawI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
- link jawS: geometry visual mesh filename=package://udg_pandora_sim/data2/robot2/NEW_PANDORA_ARM/jawS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
- link palm: geometry visual mesh filename=package://udg_pandora_sim/data2/robot2/NEW_PANDORA_ARM/part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
- link shoulder: geometry visual mesh filename=package://udg_pandora_sim/data2/robot2/NEW_PANDORA_ARM/part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

File: udg_pandora_sim/scenes/valvePanel.urdf (robot description, URDF)
Before this commit: robot valvePanel, 2 links, 1 joints
Links:
- link bar: geometry visual mesh filename=package://udg_pandora_sim/data2/objects2/handle.osg
- link handle: geometry visual mesh filename=package://udg_pandora_sim/data2/objects2/handle.osg
