Commit message: Add jaw in G500Arm.urdf model and chage load_manifest in sim_link_detector

File: udg_pandora_sim/config/g500ARM.urdf (robot description, URDF)
Before this commit: robot girona500, 6 links, 5 joints
Links:
- added link jaw; visual mesh filename=package://udg_pandora_sim/data2/robot2/NEW_PANDORA_ARM/bb_j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
Joints:
- added joint palm_to_jawS: type fixed, parent palm, child jaw, origin xyz=0.08 -0.03 0.0 rpy=0 0 0.0, axis 0 0 1
